File: src/ESP32LAN/KiCad/esp32-ethernet.sch (KiCad schematic (older format))
At the start: 19 parts, among them IC1 BME280, IC2 ESP-WROOM-32, IC3 NCP1117-3.3, J1 SERIAL, J2 POWER, J3 IO1, J4 IO2, Y1 SG5032CAN 50MHz

Commit message: fix add more files
Parts:
- C1, C11, C2, C3: symbol C -> esp32-ethernet-rescue:C
- IC1: symbol BME280 -> esp32-ethernet-rescue:BME280
- IC2: symbol ESP-WROOM-32 -> esp32-ethernet-rescue:ESP-WROOM-32
- IC3: symbol LM1117-3.3 -> esp32-ethernet-rescue:LM1117-3.3
- J1: symbol CONN_01x06 -> esp32-ethernet-rescue:CONN_01x06
- J2: symbol CONN_01x02 -> esp32-ethernet-rescue:CONN_01x02
- J3, J4: symbol CONN_01x08 -> esp32-ethernet-rescue:CONN_01x08
- JP1: symbol Jumper_NO_Small -> esp32-ethernet-rescue:Jumper_NO_Small
- R1, R2, R3, R4, R5, R6: symbol R -> esp32-ethernet-rescue:R
- Y1: symbol OSCILLATOR_4 -> esp32-ethernet-rescue:OSCILLATOR_4
Changed lines of the file:
@@
-EESchema Schematic File Version 2
-LIBS:power
-LIBS:device
-LIBS:transistors
-LIBS:conn
-LIBS:linear
-LIBS:regul
-LIBS:74xx
-LIBS:cmos4000
-LIBS:adc-dac
-LIBS:memory
-LIBS:xilinx
-LIBS:microcontrollers
-LIBS:dsp
-LIBS:analog_switches
-LIBS:motorola
-LIBS:texas
-LIBS:intel
-LIBS:audio
-LIBS:interface
-LIBS:digital-audio
-LIBS:philips
-LIBS:display
-LIBS:cypress
-LIBS:siliconi
-LIBS:opto
-LIBS:atmel
-LIBS:contrib
-LIBS:valves
-LIBS:agg-kicad
+EESchema Schematic File Version 4
 LIBS:esp32-ethernet-cache
-EELAYER 26 0
+EELAYER 30 0
 EELAYER END
 $Descr A4 11693 8268
@@
 $EndDescr
 $Comp
-L ESP-WROOM-32 IC2
+L esp32-ethernet-rescue:ESP-WROOM-32 IC2
 U 1 1 592296D2
 P 3200 2950
@@
 $EndComp
 $Comp
-L GND #PWR01
+L esp32-ethernet-rescue:GND #PWR01
 U 1 1 5924C1F7
 P 1700 2100
@@
 $EndComp
 $Comp
-L 3v3 #PWR02
+L esp32-ethernet-rescue:3v3 #PWR02
 U 1 1 5924C2DA
 P 1950 1750
@@
 PHY_CLK
 $Comp
-L R R3
+L esp32-ethernet-rescue:R R3
 U 1 1 5924BFC1
 P 4300 1600
@@
 $EndComp
 $Comp
-L 3v3 #PWR03
+L esp32-ethernet-rescue:3v3 #PWR03
 U 1 1 5924C111
 P 4300 1350
@@
 $EndComp
 $Comp
-L OSCILLATOR_4 Y1
+L esp32-ethernet-rescue:OSCILLATOR_4 Y1
 U 1 1 5924C512
 P 10300 2950
@@
 PHY_CLK_EN
 $Comp
-L R R6
+L esp32-ethernet-rescue:R R6
 U 1 1 5924C9EB
 P 9850 2500
@@
 $EndComp
 $Comp
-L GND #PWR04
+L esp32-ethernet-rescue:GND #PWR04
 U 1 1 5924CBB2
 P 9850 2300
@@
 PHY_CLK_EN
 $Comp
-L GND #PWR05
+L esp32-ethernet-rescue:GND #PWR05
 U 1 1 5924CEF7
 P 10850 2650
@@
 $EndComp
 $Comp
-L 3v3 #PWR06
+L esp32-ethernet-rescue:3v3 #PWR06
 U 1 1 5924D080
 P 10850 3150
@@
 Power Budget @ 3.3V:\nESP-WROOM-32: 260mA\nLAN8720A: 54mA\n\nTotal: approx 350mA
 $Comp
-L C C2
+L esp32-ethernet-rescue:C C2
 U 1 1 59257C30
 P 9500 1300
@@
 $EndComp
 $Comp
-L LM1117-3.3 IC3
+L esp32-ethernet-rescue:LM1117-3.3 IC3
 U 1 1 59257F22
 P 10050 1050
@@
 $EndComp
 $Comp
-L GND #PWR07
+L esp32-ethernet-rescue:GND #PWR07
 U 1 1 592580C8
 P 9500 1550
@@
 $EndComp
 $Comp
-L GND #PWR08
+L esp32-ethernet-rescue:GND #PWR08
 U 1 1 59258178
 P 10050 1550
@@
 $EndComp
 $Comp
-L GND #PWR09
+L esp32-ethernet-rescue:GND #PWR09
 U 1 1 59258228
 P 10600 1550
@@
 $EndComp
 $Comp
-L 3v3 #PWR010
+L esp32-ethernet-rescue:3v3 #PWR010
 U 1 1 592583D5
 P 10600 850
@@
 $EndComp
 $Comp
-L C C3
+L esp32-ethernet-rescue:C C3
 U 1 1 59258465
 P 10600 1300
@@
 $EndComp
 $Comp
-L CONN_01x02 J2
+L esp32-ethernet-rescue:CONN_01x02 J2
 U 1 1 59258CB6
 P 8800 1100
@@
 $EndComp
 $Comp
-L CONN_01x06 J1
+L esp32-ethernet-rescue:CONN_01x06 J1
 U 1 1 5925A0F7
 P 1100 2450
@@
 FTDI pinout:\n1 - BLK - GND\n2 - BRN - CTS#\n3 - RED - VCC\n4 - ORG - TXD\n5 - YEL - RXD\n6 - GRN - RTS#
 $Comp
-L GND #PWR011
+L esp32-ethernet-rescue:GND #PWR011
 U 1 1 5925A328
 P 1550 2450
@@
 $EndComp
 $Comp
-L 3v3 #PWR012
+L esp32-ethernet-rescue:3v3 #PWR012
 U 1 1 5925B3DF
 P 1700 2600
@@
 NoConn ~ 1200 2550
 $Comp
-L Jumper_NO_Small JP1
+L esp32-ethernet-rescue:Jumper_NO_Small JP1
 U 1 1 5925BC6A
 P 4850 1600
@@
 $EndComp
 $Comp
-L GND #PWR013
+L esp32-ethernet-rescue:GND #PWR013
 U 1 1 5925C082
 P 4850 1400
@@
 PHY_CLK
 $Comp
-L R R4
+L esp32-ethernet-rescue:R R4
 U 1 1 5925DD16
 P 5250 1850
@@
 $EndComp
 $Comp
-L BME280 IC1
+L esp32-ethernet-rescue:BME280 IC1
 U 1 1 592AD5C5
 P 2350 5900
@@
 $EndComp
 $Comp
-L GND #PWR014
+L esp32-ethernet-rescue:GND #PWR014
 U 1 1 592AD7A0
 P 1900 6150
@@
 $EndComp
 $Comp
-L C C1
+L esp32-ethernet-rescue:C C1
 U 1 1 592AD97F
 P 1750 5950
@@
 $EndComp
 $Comp
-L 3v3 #PWR015
+L esp32-ethernet-rescue:3v3 #PWR015
 U 1 1 592AE1D3
 P 1750 5650
@@
 $EndComp
 $Comp
-L GND #PWR016
+L esp32-ethernet-rescue:GND #PWR016
 U 1 1 592AE7A8
 P 3150 6000
@@
 $EndComp
 $Comp
-L R R1
+L esp32-ethernet-rescue:R R1
 U 1 1 592ADD44
 P 2850 5550
@@
 $EndComp
 $Comp
-L R R2
+L esp32-ethernet-rescue:R R2
 U 1 1 592ADDFE
 P 3200 5550
@@
 I2C_SDA
 $Comp
-L 3v3 #PWR017
+L esp32-ethernet-rescue:3v3 #PWR017
 U 1 1 592AE9EC
 P 3000 5250
@@
 	2850 5700 2850 5800
 Wire Wire Line
-	3350 5900 2750 5900
-Wire Wire Line
-	3350 5800 2750 5800
+	3350 5900 3200 5900
+Wire Wire Line
+	3350 5800 2850 5800
 Connection ~ 2850 5400
 Wire Wire Line
-	2750 5400 3200 5400
+	2750 5400 2850 5400
 Wire Wire Line
 	2750 5400 2750 5700
@@
 	1750 6100 1900 6100
 Wire Wire Line
-	1750 5800 1950 5800
+	1750 5800 1900 5800
 Connection ~ 1900 6100
 Connection ~ 1900 5800
@@
 	1900 5900 1950 5900
 Wire Wire Line
-	1900 5900 1900 6150
+	1900 5900 1900 6000
 Wire Wire Line
 	5400 1850 5450 1850
 Wire Wire Line
-	4200 1850 5100 1850
+	4200 1850 4300 1850
 Wire Wire Line
 	9800 2950 9900 2950
@@
 	1200 2450 1550 2450
 Wire Wire Line
-	8900 1100 9500 1100
+	8900 1100 9200 1100
 Wire Wire Line
 	8950 1200 8900 1200
@@
 	8950 1550 8950 1200
 Wire Wire Line
-	9500 1550 8950 1550
+	9500 1550 9150 1550
 Connection ~ 9500 1100
 Wire Wire Line
 	9500 1050 9750 1050
 Wire Wire Line
-	9500 1050 9500 1150
+	9500 1050 9500 1100
 Connection ~ 10600 1050
 Wire Wire Line
-	10600 850  10600 1150
+	10600 850  10600 1050
 Wire Wire Line
 	10350 1050 10600 1050
@@
 	4200 2350 5800 2350
 Wire Wire Line
-	9800 2850 9900 2850
+	9800 2850 9850 2850
 Wire Wire Line
 	9850 2350 9850 2300
@@
 	1700 2100 2200 2100
 Wire Wire Line
-	2200 1950 2200 2250
+	2200 1950 2200 2050
 Wire Wire Line
 	5800 3150 5800 3000
@@
 PHY_CLK
 $Comp
-L R R5
+L esp32-ethernet-rescue:R R5
 U 1 1 592B44E5
 P 7650 2500
@@
 	4200 3750 4450 3750
 $Comp
-L 3v3 #PWR018
+L esp32-ethernet-rescue:3v3 #PWR018
 U 1 1 592B8566
 P 5950 5000
@@
 	5950 5100 5950 5000
 $Comp
-L GND #PWR019
+L esp32-ethernet-rescue:GND #PWR019
 U 1 1 592B8700
 P 5950 5850
@@
 	5850 5500 6000 5500
 $Comp
-L CONN_01x08 J3
+L esp32-ethernet-rescue:CONN_01x08 J3
 U 1 1 592B9758
 P 5750 5100
@@
 	5850 5700 6000 5700
 $Comp
-L CONN_01x08 J4
+L esp32-ethernet-rescue:CONN_01x08 J4
 U 1 1 592B9F34
 P 6600 5100
@@
 	6700 5700 6850 5700
 $Comp
-L GND #PWR020
+L esp32-ethernet-rescue:GND #PWR020
 U 1 1 592AE7FC
 P 6850 5850
@@
 	6850 5800 6850 5850
 $Comp
-L PWR #FLG021
+L esp32-ethernet-rescue:PWR #FLG021
 U 1 1 592AEC20
 P 9200 1000
@@
 $EndComp
 $Comp
-L PWR #FLG022
+L esp32-ethernet-rescue:PWR #FLG022
 U 1 1 592AECE0
 P 9150 1650
@@
 Connection ~ 9150 1550
 $Comp
-L C C11
+L esp32-ethernet-rescue:C C11
 U 1 1 592B0E6B
 P 10850 2900
@@
 Wire Wire Line
 	10850 3050 10850 3150
+Wire Wire Line
+	9850 2850 9900 2850
+Wire Wire Line
+	3000 5400 3200 5400
+Wire Wire Line
+	3200 5900 2750 5900
+Wire Wire Line
+	2850 5800 2750 5800
+Wire Wire Line
+	2850 5400 3000 5400
+Wire Wire Line
+	1900 6100 1900 6150
+Wire Wire Line
+	1900 5800 1950 5800
+Wire Wire Line
+	1900 6000 1900 6100
+Wire Wire Line
+	4850 1850 5100 1850
+Wire Wire Line
+	9500 1100 9500 1150
+Wire Wire Line
+	10600 1050 10600 1150
+Wire Wire Line
+	4300 1850 4850 1850
+Wire Wire Line
+	2200 2150 2200 2250
+Wire Wire Line
+	2200 2050 2200 2150
+Wire Wire Line
+	9200 1100 9500 1100
+Wire Wire Line
+	9150 1550 8950 1550
 $EndSCHEMATC
